Commit message: feed dispersion mapper rewrite

File: matsyota_ws/src/matsyota_simulator/urdf/asv.urdf.xacro (robot description, xacro)
@@ -2,4 +2,11 @@
 <robot name="matsyota_asv" xmlns:xacro="http://ros.org/wiki/xacro">
   <xacro:arg name="namespace" default="asv"/>
+  <!-- Dummy root link to avoid KDL inertia error -->
+  <link name="$(arg namespace)/base_footprint" />
+  <joint name="$(arg namespace)/base_joint" type="fixed">
+    <parent link="$(arg namespace)/base_footprint" />
+    <child link="$(arg namespace)/base_link" />
+    <origin xyz="0 0 0" rpy="0 0 0" />
+  </joint>
   <link name="$(arg namespace)/base_link">
     <visual>
